Commit message: three robot in map without explore

File: src/robotics_project_pkg/urdf/limo_four_diff.xacro (robot description, xacro)
@@ -1,6 +1,10 @@
 <?xml version="1.0"?>
 <robot name="limo_four_diff" xmlns:xacro="http://ros.org/wiki/xacro">
-    <xacro:include filename="$(find limo_description)/urdf/limo_xacro.xacro" />
-    <xacro:include filename="$(find limo_description)/urdf/limo_four_diff.gazebo" />
+    <xacro:arg name="robot_namespace" default="robot"/>
+    <!-- Expose namespace as property for included files -->
+    <xacro:property name="ns" value="$(arg robot_namespace)"/>
+    <!-- 2. Include other Xacro files -->
+    <xacro:include filename="$(find robotics_project_pkg)/urdf/limo_xacro.xacro" />
+    <xacro:include filename="$(find robotics_project_pkg)/urdf/limo_four_diff.gazebo" />
     <!-- Variables -->
     <xacro:property name="M_PI" value="3.14159"/>
@@ -15,12 +19,13 @@
     <xacro:property name="wheel_length" value="0.045" />
     <xacro:property name="wheel_radius" value="0.045" />
-  <link name="base_footprint"/>
-  <joint name="base_joint" type="fixed">
-    <parent link="base_footprint"/>
-    <child link="base_link"/>
-    <origin xyz="0.0 0.0 0.15" rpy="0 0 0"/>
-  </joint>
+    <!-- Base footprint -->
+    <link name="${ns}_base_footprint"/>
+    <joint name="${ns}_base_joint" type="fixed">
+        <parent link="${ns}_base_footprint"/>
+        <child link="${ns}_base_link"/>
+        <origin xyz="0.0 0.0 0.15" rpy="0 0 0"/>
+    </joint>
     <!-- Base link -->
-    <link name="base_link">
+    <link name="${ns}_base_link">
         <visual>
             <origin xyz="0 0 -0.15" rpy="0 0 1.57" />
@@ -30,12 +35,12 @@
         </visual>
         <collision>
-            <!--origin xyz="0 0 -0.15" rpy="0 0 1.57" /-->
             <origin xyz="0 0 0" rpy="0 0 0" />
-          <geometry>
-              <box size="${base_x_size} ${base_y_size} ${base_z_size}"/>
-          </geometry>
+            <geometry>
+                <box size="${base_x_size} ${base_y_size} ${base_z_size}"/>
+            </geometry>
         </collision>
     </link>
-    <link name="inertial_link">
+    <!-- Inertial -->
+    <link name="${ns}_inertial_link">
         <inertial>
             <origin xyz="0.0 0.0 0.0" />
@@ -46,28 +51,32 @@
         </inertial>
     </link>
-    <joint name="inertial_joint" type="fixed">
+    <joint name="${ns}_inertial_joint" type="fixed">
         <origin xyz="0 0 0" rpy="0 0 0" />
-        <parent link="base_link" />
-        <child link="inertial_link" />
+        <parent link="${ns}_base_link" />
+        <child link="${ns}_inertial_link" />
     </joint>
-    <xacro:limo_laser parent_prefix="base_link" frame_prefix="laser">
+    <!-- Laser -->
+    <xacro:limo_laser parent_prefix="${ns}_base_link" frame_prefix="${ns}_laser">
         <origin xyz="0.103 0 -0.034" rpy="0 0 0"/>
     </xacro:limo_laser>
-    <xacro:limo_depth_camera parent_prefix="base_link" frame_prefix="depth_camera">
+    <!-- Depth camera -->
+    <xacro:limo_depth_camera parent_prefix="${ns}_base_link" frame_prefix="${ns}_depth_camera">
         <origin xyz="0.084 0 0.03" rpy="0 0 0"/>
     </xacro:limo_depth_camera>
-    <xacro:limo_imu parent_prefix="base_link" frame_prefix="imu">
+    <!-- IMU -->
+    <xacro:limo_imu parent_prefix="${ns}_base_link" frame_prefix="${ns}_imu">
         <origin xyz="0.0 0 -0.1" rpy="0 0 0"/>
     </xacro:limo_imu>
-    <xacro:limo_wheel parent_prefix="base_link" wheel_prefix="front_left" reflect="1">
-        <origin xyz="${wheelbase/2} ${track/2} ${wheel_vertical_offset}" rpy="0 0  0" />
+    <!-- Wheels -->
+    <xacro:limo_wheel parent_prefix="${ns}_base_link" wheel_prefix="${ns}_front_left" reflect="1">
+        <origin xyz="${wheelbase/2} ${track/2} ${wheel_vertical_offset}" rpy="0 0 0" />
     </xacro:limo_wheel>
-    <xacro:limo_wheel parent_prefix="base_link" wheel_prefix="front_right" reflect="-1">
+    <xacro:limo_wheel parent_prefix="${ns}_base_link" wheel_prefix="${ns}_front_right" reflect="-1">
         <origin xyz="${wheelbase/2} ${-track/2} ${wheel_vertical_offset}" rpy="${M_PI} 0 0" />
     </xacro:limo_wheel>
-    <xacro:limo_wheel parent_prefix="base_link" wheel_prefix="rear_left" reflect="1">
+    <xacro:limo_wheel parent_prefix="${ns}_base_link" wheel_prefix="${ns}_rear_left" reflect="1">
         <origin xyz="${-wheelbase/2} ${track/2} ${wheel_vertical_offset}" rpy="0 0 0" />
     </xacro:limo_wheel>
-    <xacro:limo_wheel parent_prefix="base_link" wheel_prefix="rear_right" reflect="-1">
+    <xacro:limo_wheel parent_prefix="${ns}_base_link" wheel_prefix="${ns}_rear_right" reflect="-1">
         <origin xyz="${-wheelbase/2} ${-track/2} ${wheel_vertical_offset}" rpy="${M_PI} 0 0" />
     </xacro:limo_wheel>

File: src/robotics_project_pkg/urdf/limo_xacro.xacro (robot description, xacro)
@@ -1,4 +1,6 @@
 <?xml version="1.0"?>
 <robot name="limo_xacro" xmlns:xacro="http://ros.org/wiki/xacro">
+    <xacro:arg name="robot_namespace" default="robot"/>
+    <xacro:property name="ns" value="$(arg robot_namespace)"/>
     <xacro:macro name="limo_wheel" params="parent_prefix wheel_prefix reflect *joint_pose">
         <link name="${wheel_prefix}_wheel_link">
@@ -59,5 +61,5 @@
             </collision>
         </link>
-        <joint type="fixed" name="laser_joint">
+        <joint type="fixed" name="${frame_prefix}_joint">
             <xacro:insert_block name="joint_pose"/>
             <child link="${frame_prefix}_link"/>
@@ -99,14 +101,14 @@
             </collision>
         </link>
-        <joint type="fixed" name="depth_camera_joint">
+        <joint type="fixed" name="${frame_prefix}_joint">
             <xacro:insert_block name="joint_pose"/>
             <child link="${frame_prefix}_link"/>
             <parent link="${parent_prefix}"/>
         </joint>
-        <link name="depth_link"></link>
+        <link name="${frame_prefix}_depth_link"></link>
         <joint name="${frame_prefix}_to_camera_joint" type="fixed">
             <origin xyz="0 0 0" rpy="${-M_PI/2} 0 ${-M_PI/2} "/>
             <parent link="${frame_prefix}_link"/>
-            <child link="depth_link"/>
+            <child link="${frame_prefix}_depth_link"/>
           </joint>
         <gazebo reference="${frame_prefix}_link">
@@ -145,5 +147,5 @@
             </collision>
         </link>
-        <joint type="fixed" name="imu_joint">
+        <joint type="fixed" name="${frame_prefix}_joint">
             <xacro:insert_block name="joint_pose"/>
             <child link="${frame_prefix}_link"/>

Commit message: visual robots

File: src/robotics_project_pkg/urdf/limo_four_diff.xacro (robot description, xacro)
@@ -4,5 +4,5 @@
     <!-- Expose namespace as property for included files -->
     <xacro:property name="ns" value="$(arg robot_namespace)"/>
-    <!-- 2. Include other Xacro files -->
+    <!-- Include other Xacro files -->
     <xacro:include filename="$(find robotics_project_pkg)/urdf/limo_xacro.xacro" />
     <xacro:include filename="$(find robotics_project_pkg)/urdf/limo_four_diff.gazebo" />
@@ -19,13 +19,18 @@
     <xacro:property name="wheel_length" value="0.045" />
     <xacro:property name="wheel_radius" value="0.045" />
+    <!--
+    CRITICAL: Link names are now GENERIC (no namespace prefix)
+    The tf_prefix parameter in robot_state_publisher will add the namespace
+    Example: base_footprint becomes robot1/base_footprint in TF
+    -->
     <!-- Base footprint -->
-    <link name="${ns}_base_footprint"/>
-    <joint name="${ns}_base_joint" type="fixed">
-        <parent link="${ns}_base_footprint"/>
-        <child link="${ns}_base_link"/>
+    <link name="base_footprint"/>
+    <joint name="base_joint" type="fixed">
+        <parent link="base_footprint"/>
+        <child link="base_link"/>
         <origin xyz="0.0 0.0 0.15" rpy="0 0 0"/>
     </joint>
     <!-- Base link -->
-    <link name="${ns}_base_link">
+    <link name="base_link">
         <visual>
             <origin xyz="0 0 -0.15" rpy="0 0 1.57" />
@@ -41,6 +46,6 @@
         </collision>
     </link>
-    <!-- Inertial -->
-    <link name="${ns}_inertial_link">
+    <!-- Inertial link -->
+    <link name="inertial_link">
         <inertial>
             <origin xyz="0.0 0.0 0.0" />
@@ -51,32 +56,32 @@
         </inertial>
     </link>
-    <joint name="${ns}_inertial_joint" type="fixed">
+    <joint name="inertial_joint" type="fixed">
         <origin xyz="0 0 0" rpy="0 0 0" />
-        <parent link="${ns}_base_link" />
-        <child link="${ns}_inertial_link" />
+        <parent link="base_link" />
+        <child link="inertial_link" />
     </joint>
-    <!-- Laser -->
-    <xacro:limo_laser parent_prefix="${ns}_base_link" frame_prefix="${ns}_laser">
+    <!-- Laser sensor - generic names -->
+    <xacro:limo_laser parent_prefix="base_link" frame_prefix="laser">
         <origin xyz="0.103 0 -0.034" rpy="0 0 0"/>
     </xacro:limo_laser>
-    <!-- Depth camera -->
-    <xacro:limo_depth_camera parent_prefix="${ns}_base_link" frame_prefix="${ns}_depth_camera">
+    <!-- Depth camera - generic names -->
+    <xacro:limo_depth_camera parent_prefix="base_link" frame_prefix="depth_camera">
         <origin xyz="0.084 0 0.03" rpy="0 0 0"/>
     </xacro:limo_depth_camera>
-    <!-- IMU -->
-    <xacro:limo_imu parent_prefix="${ns}_base_link" frame_prefix="${ns}_imu">
+    <!-- IMU sensor - generic names -->
+    <xacro:limo_imu parent_prefix="base_link" frame_prefix="imu">
         <origin xyz="0.0 0 -0.1" rpy="0 0 0"/>
     </xacro:limo_imu>
-    <!-- Wheels -->
-    <xacro:limo_wheel parent_prefix="${ns}_base_link" wheel_prefix="${ns}_front_left" reflect="1">
+    <!-- Wheels - generic names -->
+    <xacro:limo_wheel parent_prefix="base_link" wheel_prefix="front_left" reflect="1">
         <origin xyz="${wheelbase/2} ${track/2} ${wheel_vertical_offset}" rpy="0 0 0" />
     </xacro:limo_wheel>
-    <xacro:limo_wheel parent_prefix="${ns}_base_link" wheel_prefix="${ns}_front_right" reflect="-1">
+    <xacro:limo_wheel parent_prefix="base_link" wheel_prefix="front_right" reflect="-1">
         <origin xyz="${wheelbase/2} ${-track/2} ${wheel_vertical_offset}" rpy="${M_PI} 0 0" />
     </xacro:limo_wheel>
-    <xacro:limo_wheel parent_prefix="${ns}_base_link" wheel_prefix="${ns}_rear_left" reflect="1">
+    <xacro:limo_wheel parent_prefix="base_link" wheel_prefix="rear_left" reflect="1">
         <origin xyz="${-wheelbase/2} ${track/2} ${wheel_vertical_offset}" rpy="0 0 0" />
     </xacro:limo_wheel>
-    <xacro:limo_wheel parent_prefix="${ns}_base_link" wheel_prefix="${ns}_rear_right" reflect="-1">
+    <xacro:limo_wheel parent_prefix="base_link" wheel_prefix="rear_right" reflect="-1">
         <origin xyz="${-wheelbase/2} ${-track/2} ${wheel_vertical_offset}" rpy="${M_PI} 0 0" />
     </xacro:limo_wheel>
